Commit message: Adicionando joint+link RViz

File: urdf/robot.urdf (robot description, URDF)
Before this commit: robot m2wr, 1 links, 0 joints
Links:
- added link right_wheel, mass 0.2; collision cylinder length=0.04 radius=0.1; visual cylinder length=0.04 radius=0.1
Joints:
- added joint joint_right_wheel: type continuous, parent chassis, child right_wheel, origin xyz=-0.15 -0.15 0 rpy=0 0 0, axis 0 1 0, limit effort=10000 velocity=1000

Commit message: dummy link

File: urdf/robot.urdf (robot description, URDF)
Before this commit: robot m2wr, 2 links, 1 joints
Links:
- added link dummy
Joints:
- added joint dummy_joint: type fixed, parent dummy, child chassis
