Commit message: Add camera

File: urdf/plugins.xacro (robot description, xacro)
@@ -25,3 +25,40 @@
     </plugin>
   </gazebo>
+  <gazebo reference="link_camera">
+    <material>Gazebo/Red</material>
+    <sensor type="camera" name="camera1">
+      <update_rate>30.0</update_rate>
+      <camera name="head">
+        <horizontal_fov>1.3962634</horizontal_fov>
+        <image>
+          <width>800</width>
+          <height>800</height>
+          <format>R8G8B8</format>
+        </image>
+        <clip>
+          <near>0.02</near>
+          <far>300</far>
+        </clip>
+        <noise>
+          <type>gaussian</type>
+          <mean>0.0</mean>
+          <stddev>0.007</stddev>
+        </noise>
+      </camera>
+      <plugin name="camera_controller" filename="libgazebo_ros_camera.so">
+        <alwaysOn>true</alwaysOn>
+        <updateRate>0.0</updateRate>
+        <cameraName>rrbot/camera1</cameraName>
+        <imageTopicName>image_raw</imageTopicName>
+        <cameraInfoTopicName>camera_info</cameraInfoTopicName>
+        <frameName>link_camera</frameName>
+        <hackBaseline>0.07</hackBaseline>
+        <distortionK1>0.0</distortionK1>
+        <distortionK2>0.0</distortionK2>
+        <distortionK3>0.0</distortionK3>
+        <distortionT1>0.0</distortionT1>
+        <distortionT2>0.0</distortionT2>
+      </plugin>
+    </sensor>
+  </gazebo>
 </robot>

File: urdf/robot.xacro (robot description, xacro)
@@ -1,7 +1,8 @@
 <?xml version="1.0" ?>
 <robot name="robot" xmlns:xacro="http://www.ros.org/wiki/xacro">
-  <xacro:include filename="$(find robot_description)/urdf/wheel.xacro" />
+  <xacro:include filename="$(find robot_description)/urdf/camera.xacro" />
   <xacro:include filename="$(find robot_description)/urdf/caster.xacro" />
   <xacro:include filename="$(find robot_description)/urdf/plugins.xacro" />
+  <xacro:include filename="$(find robot_description)/urdf/wheel.xacro" />
   <!-- Dummy -->
   <link name="dummy"></link>
@@ -37,3 +38,5 @@
   <!-- Caster -->
   <xacro:caster_sphere name="caster" diameter="0.1" origin="0.20 0 -0.05" />
+  <!-- Camera -->
+  <xacro:camera joint="joint_chassis_camera" link="link_camera" parent="chassis" />
 </robot>
