Commit message: xacro - propriedades e launch file

File: urdf/robot.xacro (robot description, xacro)
@@ -6,9 +6,11 @@
     <child link="chassis" />
   </joint>
+  <xacro:property name="chassis_mass" value="5.0" />
+  <xacro:property name="chassis_size" value="0.5 0.3 0.07" />
   <link name="chassis">
     <!-- pose and inertial -->
     <pose>0 0 0.1 0 0 0</pose>
     <inertial>
-      <mass value="5"/>
+      <mass value="${chassis_mass}" />
       <origin rpy="0 0 0" xyz="0 0 0.1"/>
       <inertia ixx="0.0395416666667" ixy="0" ixz="0" iyy="0.106208333333" iyz="0" izz="0.106208333333"/>
@@ -16,5 +18,5 @@
     <collision>
       <geometry>
-        <box size="0.5 0.3 0.07"/>
+        <box size="${chassis_size}" />
       </geometry>
     </collision>
@@ -22,5 +24,5 @@
       <origin rpy="0 0 0" xyz="0 0 0"/>
       <geometry>
-        <box size="0.5 0.3 0.07"/>
+        <box size="${chassis_size}"/>
       </geometry>
     </visual>

Commit message: xacro - include

File: urdf/robot.xacro (robot description, xacro)
@@ -1,4 +1,6 @@
 <?xml version="1.0" ?>
 <robot name="m2wr" xmlns:xacro="http://www.ros.org/wiki/xacro">>
+  <xacro:include filename="$(find robot_description)/urdf/wheel.xacro" />
+  <!-- Dummy -->
   <link name="dummy"></link>
   <joint name="dummy_joint" type="fixed">
@@ -28,30 +30,5 @@
     </visual>
   </link>
-  <link name="right_wheel">
-    <inertial>
-      <mass value="0.2"/>
-      <origin rpy="0 1.5707 1.5707" xyz="0 0 0"/>
-      <inertia ixx="0.000526666666667" ixy="0" ixz="0" iyy="0.000526666666667" iyz="0" izz="0.001"/>
-    </inertial>
-    <collision>
-      <origin rpy="0 1.5707 1.5707" xyz="0 0 0"/>
-      <geometry>
-        <cylinder length="0.04" radius="0.1"/>
-      </geometry>
-    </collision>
-    <visual>
-      <origin rpy="0 1.5707 1.5707" xyz="0 0 0"/>
-      <geometry>
-        <cylinder length="0.04" radius="0.1"/>
-      </geometry>
-    </visual>
-  </link>
-  <joint name="joint_right_wheel" type="continuous">
-    <origin rpy="0 0 0" xyz="-0.15 -0.15 0"/>
-    <child link="right_wheel"/>
-    <parent link="chassis"/>
-    <axis rpy="0 0 0" xyz="0 1 0"/>
-    <limit effort="10000" velocity="1000"/>
-    <joint_properties damping="1.0" friction="1.0"/>
-  </joint>
+  <!-- Wheels -->
+  <xacro:wheel name="right" />
 </robot>

Commit message: xacro - expressao matematica

File: urdf/robot.xacro (robot description, xacro)
@@ -31,4 +31,4 @@
   </link>
   <!-- Wheels -->
-  <xacro:wheel name="right" />
+  <xacro:wheel name="right" diameter="0.2" />
 </robot>

File: urdf/wheel.xacro (robot description, xacro)
@@ -1,5 +1,5 @@
 <?xml version="1.0" ?>
 <robot xmlns:xacro="http://www.ros.org/wiki/xacro">
-  <xacro:macro name="wheel" params="name">
+  <xacro:macro name="wheel" params="name diameter">
     <link name="${name}_wheel">
       <inertial>
@@ -11,5 +11,5 @@
         <origin rpy="0 1.5707 1.5707" xyz="0 0 0"/>
         <geometry>
-          <cylinder length="0.04" radius="0.1"/>
+          <cylinder length="0.04" radius="${diameter/2}"/>
         </geometry>
       </collision>
@@ -17,5 +17,5 @@
         <origin rpy="0 1.5707 1.5707" xyz="0 0 0"/>
         <geometry>
-          <cylinder length="0.04" radius="0.1"/>
+          <cylinder length="0.04" radius="${diameter/2}"/>
         </geometry>
       </visual>

Commit message: xacro if conditional

File: urdf/robot.xacro (robot description, xacro)
@@ -31,4 +31,5 @@
   </link>
   <!-- Wheels -->
-  <xacro:wheel name="right" diameter="0.2" />
+  <xacro:wheel right="1" name="right" diameter="0.2" />
+  <xacro:wheel right="0" name="left" diameter="0.2" />
 </robot>

File: urdf/wheel.xacro (robot description, xacro)
@@ -1,5 +1,5 @@
 <?xml version="1.0" ?>
 <robot xmlns:xacro="http://www.ros.org/wiki/xacro">
-  <xacro:macro name="wheel" params="name diameter">
+  <xacro:macro name="wheel" params="name diameter right">
     <link name="${name}_wheel">
       <inertial>
@@ -22,5 +22,10 @@
     </link>
     <joint name="joint_${name}_wheel" type="continuous">
-      <origin rpy="0 0 0" xyz="-0.15 -0.15 0"/>
+      <xacro:if value="${right == 1}">
+        <origin rpy="0 0 0" xyz="-0.15 -0.15 0" />
+      </xacro:if>
+      <xacro:if value="${right == 0}">
+        <origin rpy="0 0 0" xyz="-0.15 0.15 0" />
+      </xacro:if>
       <child link="${name}_wheel"/>
       <parent link="chassis"/>

Commit message: caster back + fix drift issue

File: urdf/robot.xacro (robot description, xacro)
@@ -37,5 +37,6 @@
   <xacro:wheel right="0" name="left" diameter="0.2" />
   <!-- Caster -->
-  <xacro:caster_sphere name="caster" diameter="0.1" origin="0.20 0 -0.05" />
+  <xacro:caster_sphere name="caster" diameter="0.1" origin="-0.20 0 -0.05" />
+  <xacro:caster_sphere name="caster_back" diameter="0.1" origin="0.20 0 -0.05" />
   <!-- Camera -->
   <xacro:camera joint="joint_chassis_camera" link="link_camera" parent="chassis" />

File: urdf/wheel.xacro (robot description, xacro)
@@ -26,8 +26,8 @@
     <joint name="joint_${name}_wheel" type="continuous">
       <xacro:if value="${right == 1}">
-        <origin rpy="0 0 0" xyz="-0.15 -0.15 0" />
+        <origin rpy="0 0 0" xyz="0 -0.15 0" />
       </xacro:if>
       <xacro:if value="${right == 0}">
-        <origin rpy="0 0 0" xyz="-0.15 0.15 0" />
+        <origin rpy="0 0 0" xyz="0 0.15 0" />
       </xacro:if>
       <child link="${name}_wheel"/>
